File: stopwatchy.kicad_pcb (KiCad board)
At the start: 4 copper layers, 70 x 97 mm, 82 parts, among them J1 USB_C_Receptacle_USB2.0_16P, J2 PINHD_1x4_Female, J4 PROG, Q1 DMG3415U, SW4 BTN_3, SW5 BTN_1, SW6 BTN_2, SW7 BTN_4, U1 W25Q128JVS, U3 NHD-2.4-240320CF-BSXV-F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

Commit message: Fix
Connections:
- R17 pad 1: +3V3 -> GND
Routing:
- net +3V3: track 144.0 -> 140.4 mm
Changed lines of the file:
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@@
 			(layers "B.Cu" "B.Paste" "B.Mask")
 			(roundrect_rratio 0.25)
-			(net 76 "+3V3")
+			(net 1 "GND")
 			(pintype "passive")
 		)
@@
 	)
 	(segment
-		(start 151.598445 42.63028)
-		(end 151.598445 41.652112)
-		(width 0.5)
-		(layer "B.Cu")
-		(net 76)
-	)
-	(segment
 		(start 136.7 102.5)
 		(end 137.148529 102.5)
@@
 	)
 	(segment
-		(start 151.671307 42.703142)
-		(end 151.598445 42.63028)
-		(width 0.5)
-		(layer "B.Cu")
-		(net 76)
-	)
-	(segment
 		(start 136.505946 102.694054)
 		(end 136.7 102.5)
@@
 		(width 0.5)
 		(layer "B.Cu")
-		(net 76)
-	)
-	(segment
-		(start 154.230055 42.703142)
-		(end 151.671307 42.703142)
-		(width 0.5)
-		(layer "B.Cu")
