File: stopwatchy.kicad_sch (KiCad schematic)
At the start: 80 parts, among them J1 USB_C_Receptacle_USB2.0_16P, J2 PINHD_1x4_Female, J4 PROG, Q1 DMG3415U, SW1 BOOT, SW2 RESET, SW4 BTN_3, SW5 BTN_1, SW6 BTN_2, SW7 BTN_4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

Commit message: Fix
Parts:
- removed R33, R34: 0R_0603, 4ms_Resistor:R_0603, symbol PCM_4ms_Resistor:0R_0603
Connections:
- net +3V3: no longer R17.1
- net GND: now also R17.1
- net USB_D+: now also J1.A6 (D+), J1.B6 (D+)
- net USB_D-: now also J1.A7 (D-), J1.B7 (D-)
